File: eagle/808_hihat.brd (EAGLE design)
At the start: 100 x 80 mm, 127 parts, among them IC1 TL072P, IC2 TL072P, Q21* BC546, Q22* BC546, Q23* BC546, Q24* BC546, Q26* BC546, Q27* BC546, Q28* BC546, Q29* BC546, Q3* BC546, Q30* BC546, Q31* BC546, Q4* BC546, Q7* BC556, Q8* BC556, U4 4584N

Commit message: replaced parts
Parts:
- removed C1, C2, C3, C4: 22p, TR808clone:C025-025X050
- removed C1*1, C4*1, C5*1: 18n, TR808clone:C035-030X60
- removed C2*1, C3*1: 10n, TR808clone:C035-025X75
- removed C5, C6: 0.1uF, TR808clone:C035-025X75
- removed C6*1: 22n, TR808clone:C035-030X60
- removed CH_OUT, OH_OUT: LSP11, solpad:LSP11
- removed D1, D2: 1N4148DO35-7, TR808clone:DO35-7
- removed Q21*, Q22*, Q23*, Q24*, Q26*, Q27*, Q28*, Q29*, Q3*, Q30*, Q31*, Q4*: BC546, transistor:TO92-CBE
- removed Q7*, Q8*: BC556, transistor:TO92-EBC
- removed R1, R2: 22K, TR808clone:0207/5V
- removed R35*1, R37*1, R39*1, R46*1, R48*1, R50*1: 120K, TR808clone:0207/5V
- removed R40*1, R41*1: 560K, TR808clone:0207/5V
- removed R42*1: 680K, TR808clone:0207/5V
- removed R43*1: 220K, TR808clone:0207/5V
- removed R44*1: 300K, TR808clone:0207/5V
- removed R45*1: 270K, TR808clone:0207/5V
- removed R53*1: 1K, TR808clone:0207/5V
- removed U4: 4584N, TR808clone:DIL14
- added CH_OUTPUT, OH_OUTPUT: AUDIO-JACK, erthenvar:ERTHENVAR-JACK-90DEG
- added CH_OUT_NORM, DIGI_NOISE, OH_OUT_NORM: 22-23-2021, con-molex:22-23-2021
- added Q1, Q10, Q11, Q12, Q2, Q3, Q4, Q5, Q6, Q7, Q8, Q9: 2N3904, 808_lt:TO92
- added Q13, Q14: 2N3906, 808_lt:TO92
- added U$2: POWER, eurorack:POWER_16
Connections:
- removed net N$12: R35*1.2, R40*1.1, U4.6
- removed net N$13: R37*1.1, R41*1.2, U4.4
- removed net N$14: R43*1.1, R46*1.2, U4.8
- removed net N$15: C5*1.P$2, R45*1.1, U4.11
- removed net N$16: C6*1.P$2, R44*1.1, U4.13
- removed net N$19: R39*1.1, R42*1.1, U4.2
- removed net N$22: C5.P$1, D1.C, R1.2
- removed net N$23: D1.A, OH_TRIG.MP
- removed net N$24: C6.P$1, D2.C, R2.2
- removed net N$26: CH_TRIG.MP, D2.A
- removed net N$27: IC2.6, IC2.7
- removed net N$583: Q30*.E, R152*.1
- removed net N$584: Q27*.E, R145*.1
- removed net N$606: Q29*.B, R140*.2
- removed net N$9: C4*1.P$2, R43*1.2, U4.9
- removed net TP1: R45*1.2, R48*1.1, U4.10
- removed net TP2: R44*1.2, R50*1.2, U4.12
- new net N$10: OH_OUTPUT.P$2, OH_OUT_NORM.1
- new net N$11: CH_OUTPUT.P$2, CH_OUT_NORM.1
- new net V+: IC1.8, IC2.8
- new net V-: IC1.4, IC2.4
- net +12V: now also Q1.1, Q2.1, Q6.1, U$2.10, U$2.9; no longer C1.1, C2.2, IC1.8, IC2.8, Q26*.C, Q29*.C, Q31*.C
- net +5V: now also U$2.11, U$2.12; no longer U4.14
- net -12V: now also U$2.1, U$2.2; no longer C3.2, C4.1, IC1.4, IC2.4
- net .: now also Q14.3, U$2.13, U$2.14; no longer Q8*.E
- net CH_OUT: now also CH_OUTPUT.P$3; no longer CH_OUT.MP
- net GND: now also CH_OUTPUT.P$1, CH_OUT_NORM.2, DIGI_NOISE.1, OH_OUTPUT.P$1, OH_OUT_NORM.2, Q10.3, Q11.3, Q12.3, Q8.3, Q9.3, U$2.3, U$2.4, U$2.5, U$2.6, U$2.7, U$2.8; no longer C1*1.P$1, C1.2, C2*1.P$1, C2.1, C3*1.P$1, C3.1, C4*1.P$1, C4.2, C5*1.P$1, C6*1.P$1, IC2.5, Q21*.E, Q22*.E, Q23*.E, Q3*.E, Q4*.E, R1.1, R2.1, R53*1.1, U4.7
- net N$17: now also Q13.3, U$1.13, U$1.14; no longer Q7*.E
- net N$18: now also OH_TRIG.MP, U$1.15, U$1.16; no longer C5.P$2
- net N$2: now also DIGI_NOISE.2; no longer R35*1.1, R37*1.2, R39*1.2, R46*1.1, R48*1.2, R50*1.1, R53*1.2
- net N$25: now also CH_TRIG.MP, U$2.15, U$2.16; no longer C6.P$2
- net N$559: now also Q12.2; no longer Q4*.B
- net N$560: now also Q14.2; no longer Q8*.B
- net N$562: now also Q12.1; no longer Q4*.C
- net N$563: now also Q14.1; no longer Q8*.C
- net N$566: now also Q11.2; no longer Q3*.B
- net N$567: now also Q13.2; no longer Q7*.B
- net N$568: now also Q11.1; no longer Q3*.C
- net N$569: now also Q13.1; no longer Q7*.C
- net N$571: now also Q7.1; no longer Q24*.C
- net N$572: now also Q7.2; no longer Q24*.B
- net N$573: now also Q7.3; no longer Q24*.E
- net N$574: now also Q8.1, Q9.1; no longer Q22*.C, Q23*.C
- net N$575: now also Q8.2; no longer Q22*.B
- net N$576: now also Q10.1; no longer Q21*.C
- net N$578: now also Q5.2; no longer Q28*.B
- net N$579: now also Q5.1; no longer Q28*.C
- net N$580: now also Q9.2; no longer Q23*.B
- net N$581: now also Q5.3; no longer Q28*.E
- net N$582: now also Q6.3; no longer Q29*.E
- net N$585: now also Q3.2; no longer Q30*.B
- net N$586: now also Q4.2; no longer Q27*.B
- net N$587: now also Q3.1; no longer Q30*.C
- net N$588: now also Q4.1; no longer Q27*.C
- net N$591: now also Q1.2; no longer Q26*.B
- net N$592: now also Q2.2; no longer Q31*.B
- net N$6: now also Q6.2, R140*.2; no longer C1*1.P$2, R40*1.2, U4.5
- net N$604: now also Q10.2; no longer Q21*.B
- net N$607: now also Q1.3; no longer Q26*.E
- net N$608: now also Q2.3; no longer Q31*.E
- net N$7: now also Q4.3, R145*.1; no longer C2*1.P$2, R41*1.1, U4.3
- net N$8: now also Q3.3, R152*.1; no longer C3*1.P$2, R42*1.2, U4.1
- net OH_OUT: now also OH_OUTPUT.P$3; no longer OH_OUT.MP
Routing:
- net GND: track 546.2 -> 433.6 mm
- net N$2: track 84.9 -> 0.00 mm
- net +12V: track 305.1 -> 277.0 mm
- net TP2: track 18.4 -> 0.00 mm
- net -12V: track 107.2 -> 89.6 mm
- net N$24: track 15.8 -> 0.00 mm
- net N$7: track 15.5 -> 0.00 mm
- net N$16: track 15.1 -> 0.00 mm
- net N$581: track 24.9 -> 9.82 mm
- net N$15: track 12.6 -> 0.00 mm
- net N$19: track 12.1 -> 0.00 mm
- net N$12: track 11.5 -> 0.00 mm
- net N$6: track 11.5 -> 0.00 mm
- net N$13: track 10.6 -> 0.00 mm
- net N$9: track 10.5 -> 0.00 mm
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