File: eagle/808_hihat.brd (EAGLE design)
At the start: 100 x 80 mm, 103 parts, among them IC1 TL072P, IC3 TL071P, Q1 2N3904, Q10 2N3904, Q11 2N3904, Q12 2N3904, Q13 2N3906, Q14 2N3906, Q2 2N3904, Q3 2N3904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

Commit message: 95pct5 ar
Routing:
- net GND: track 0.00 -> 422.0 mm
- net +12V: track 0.00 -> 349.2 mm
- net N$581: track 0.00 -> 236.3 mm
- net -12V: track 0.00 -> 93.9 mm
- net N$603: track 0.00 -> 40.8 mm
- net .: track 0.00 -> 40.4 mm
- net N$601: track 0.00 -> 34.0 mm
- net N$220: track 0.00 -> 33.6 mm
- net N$17: track 0.00 -> 31.5 mm
- net N$598: track 0.00 -> 31.0 mm
- net N$573: track 0.00 -> 30.1 mm
- net N$587: track 0.00 -> 29.1 mm
- net N$576: track 0.00 -> 23.1 mm
- net TO_HH: track 0.00 -> 22.9 mm
- net N$588: track 0.00 -> 22.2 mm
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
Commit message: routed
Parts:
- R59*1: device TR808clone:0207/5V -> TR808clone:0207/7
- moved R17* 6.35 mm to (20.3, 35.6), turned to 180 degrees
- moved C83* 3.59 mm to (83.8, 12.7)
- moved R154* 2.54 mm to (72.4, 47.0)
- moved R55*1 2.29 mm to (25.7, 73.7)
- moved C61* 1.80 mm to (91.4, 40.6), turned to 90 degrees
- moved R58*1 1.37 mm to (40.6, 65.5)
- moved R152* 1.27 mm to (38.1, 53.3)
- moved R172* 1.27 mm to (96.5, 24.1)
- moved C68* 1.14 mm to (55.6, 37.3)
- moved R134* 1.02 mm to (30.2, 22.9)
- moved C71*1 0.92 mm to (80.8, 32.5)
- moved C74* 0.76 mm to (75.4, 47.0)
- moved R12* 0.76 mm to (19.6, 43.2)
- moved R135* 0.76 mm to (32.3, 35.6)
- moved R153* 0.76 mm to (69.8, 58.9)
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Routing:
- net N$577: track 11.5 -> 78.7 mm, vias 0 -> 2
- net GND: track 422.0 -> 478.5 mm, vias 0 -> 2
- net N$600: track 16.6 -> 71.7 mm, vias 0 -> 2
- net -12V: track 93.9 -> 134.7 mm, vias 0 -> 2
- net +12V: track 349.2 -> 373.6 mm
- net N$11: track 0.00 -> 20.5 mm
- net OH_OUT: track 0.00 -> 10.2 mm
- net CH_OUT: track 0.00 -> 8.40 mm
- net N$10: track 0.00 -> 4.33 mm
- net N$601: track 34.0 -> 29.8 mm
- net N$17: track 31.5 -> 27.3 mm
- net N$567: track 11.2 -> 8.27 mm
- net N$3: track 4.60 -> 2.31 mm
- net N$375: track 16.0 -> 14.0 mm
- net TO_HH: track 22.9 -> 24.9 mm
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