File: eagle/808_hihat.sch (EAGLE design)
At the start: 101 parts, among them IC1 TL072P, IC2 TL072P, Q1 2N3904, Q10 2N3904, Q11 2N3904, Q12 2N3904, Q13 2N3906, Q14 2N3906, Q2 2N3904, Q3 2N3904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

Commit message: beginning manual layout
Parts:
- removed IC2: TL072P, linear:TL072P
- added IC3: TL071P, 808_lt:TL071P
Connections:
- net +12V: now also IC1P.V+, IC3.V+
- net -12V: now also IC1P.V-, IC3.V-
- net GND: now also IC3.+IN; no longer IC2A.+IN
- net N$4: now also IC3.-IN; no longer IC2A.-IN
- net TO_HH: now also IC3.OUT; no longer IC2A.OUT
Changed lines of the file:
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@@
 <part name="R58*1" library="TR808clone" deviceset="R-EU_" device="0207/2V" value="560R"/>
 <part name="IC1" library="linear" deviceset="TL072" device="P"/>
-<part name="IC2" library="linear" deviceset="TL072" device="P"/>
 <part name="U$1" library="eurorack" deviceset="POWER" device=""/>
 <part name="P+1" library="supply1" deviceset="+12V" device=""/>
@@
 <part name="Q13" library="808_lt" deviceset="2N3906" device=""/>
 <part name="Q14" library="808_lt" deviceset="2N3906" device=""/>
+<part name="P+5" library="supply1" deviceset="+12V" device=""/>
+<part name="P-5" library="supply1" deviceset="-12V" device=""/>
+<part name="IC3" library="808_lt" deviceset="TL071" device="P"/>
+<part name="P+13" library="supply1" deviceset="+12V" device=""/>
+<part name="P-6" library="supply1" deviceset="-12V" device=""/>
 </parts>
 <sheets>
@@
 <instance part="IC1" gate="A" x="147.32" y="48.26" rot="MR180"/>
 <instance part="IC1" gate="B" x="147.32" y="7.62" rot="MR180"/>
-<instance part="IC2" gate="A" x="27.94" y="-30.48" rot="MR180"/>
 <instance part="CH_ACCENT" gate="1" x="-53.34" y="25.4"/>
 <instance part="CH_TRIG" gate="1" x="-66.04" y="15.24" rot="R180"/>
@@
 <instance part="Q13" gate="G$1" x="-50.8" y="93.98"/>
 <instance part="Q14" gate="G$1" x="-48.26" y="5.08"/>
+<instance part="IC1" gate="P" x="93.98" y="101.6"/>
+<instance part="P+5" gate="1" x="93.98" y="111.76"/>
+<instance part="P-5" gate="1" x="93.98" y="91.44"/>
+<instance part="IC3" gate="A" x="27.94" y="-30.48" rot="MR180"/>
+<instance part="P+13" gate="1" x="33.02" y="-38.1"/>
+<instance part="P-6" gate="1" x="22.86" y="-22.86"/>
 </instances>
 <busses>
@@
 <wire x1="38.1" y1="0" x2="35.56" y2="0" width="0.1524" layer="91"/>
 <junction x="38.1" y="10.16"/>
-<pinref part="IC2" gate="A" pin="OUT"/>
+<pinref part="IC3" gate="A" pin="OUT"/>
 </segment>
 </net>
@@
 <segment>
 <pinref part="V2" gate="1" pin="GND"/>
-<pinref part="IC2" gate="A" pin="+IN"/>
 <wire x1="20.32" y1="-35.56" x2="20.32" y2="-33.02" width="0.1524" layer="91"/>
+<pinref part="IC3" gate="A" pin="+IN"/>
 </segment>
 <segment>
@@
 <pinref part="C15*1" gate="G$1" pin="1"/>
 <pinref part="R59*1" gate="G$1" pin="1"/>
-<pinref part="IC2" gate="A" pin="-IN"/>
+<pinref part="IC3" gate="A" pin="-IN"/>
 <junction x="20.32" y="-27.94"/>
 </segment>
@@
 <wire x1="-81.28" y1="30.48" x2="-81.28" y2="40.64" width="0.1524" layer="91"/>
 </segment>
+<segment>
+<pinref part="IC1" gate="P" pin="V+"/>
+<pinref part="P+5" gate="1" pin="+12V"/>
+</segment>
+<segment>
+<pinref part="IC3" gate="A" pin="V+"/>
+<wire x1="25.4" y1="-38.1" x2="25.4" y2="-40.64" width="0.1524" layer="91"/>
+<pinref part="P+13" gate="1" pin="+12V"/>
+<wire x1="25.4" y1="-40.64" x2="33.02" y2="-40.64" width="0.1524" layer="91"/>
+</segment>
 </net>
 <net name="-12V" class="0">
@@
 <wire x1="-81.28" y1="25.4" x2="-81.28" y2="10.16" width="0.1524" layer="91"/>
 </segment>
-</net>
+<segment>
+<pinref part="IC1" gate="P" pin="V-"/>
+<pinref part="P-5" gate="1" pin="-12V"/>
+</segment>
+<segment>
+<pinref part="IC3" gate="A" pin="V-"/>
+<wire x1="25.4" y1="-22.86" x2="25.4" y2="-20.32" width="0.1524" layer="91"/>
+<pinref part="P-6" gate="1" pin="-12V"/>
+<wire x1="25.4" y1="-20.32" x2="22.86" y2="-20.32" width="0.1524" layer="91"/>
+</segment>
+</net>

Commit message: parts on the board
Parts:
- R147*: device TR808clone:R-EU_0207/2V -> TR808clone:R-EU_0207/7
- R161*: device TR808clone:R-EU_0207/5V -> TR808clone:R-EU_0207/2V
Changed lines of the file:
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@@
 <part name="C68*" library="TR808clone" deviceset="C-EU" device="3.5MM_PITCH" value="1.5n"/>
 <part name="C73*" library="TR808clone" deviceset="C-EU" device="3.5MM_PITCH" value="1n"/>
-<part name="R147*" library="TR808clone" deviceset="R-EU_" device="0207/2V" value="2K7"/>
+<part name="R147*" library="TR808clone" deviceset="R-EU_" device="0207/7" value="2K7"/>
 <part name="R153*" library="rcl" deviceset="R-US_" device="0207/5V" value="2K7"/>
 <part name="R146*" library="TR808clone" deviceset="R-EU_" device="0207/5V" value="68K"/>
@@
 <part name="C79*" library="TR808clone" deviceset="C-EU" device="025-025X050" value="220p"/>
 <part name="R169*" library="TR808clone" deviceset="R-EU_" device="0207/5V" value="1K"/>
-<part name="R161*" library="TR808clone" deviceset="R-EU_" device="0207/5V" value="470K"/>
+<part name="R161*" library="TR808clone" deviceset="R-EU_" device="0207/2V" value="470K"/>
 <part name="C83*" library="TR808clone" deviceset="CPOL-EU" device="E2-5" value="33/6.3"/>
 <part name="C82*" library="TR808clone" deviceset="C-EU" device="025-025X050" value="220p"/>

Commit message: 93pct ar
Parts:
- C15*1, C68*: device TR808clone:C-EU3.5MM_PITCH -> TR808clone:C-EU050-024X044
- C67*: device TR808clone:C-EU4MM_PITCH -> TR808clone:C-EU050-024X044
- C74*: device TR808clone:C-EU3.5MM_PITCH -> TR808clone:C-EU050-025X075
- D13*, D14*: value 1N4148DO35-7 -> 1N4148DO35-10; device TR808clone:1N4148DO35-7 -> TR808clone:1N4148DO35-10
- R1*, R159*: device TR808clone:R-EU_0207/5V -> TR808clone:R-EU_0207/2V
- R11*, R12*, R133*, R134*, R142*, R145*, R146*, R156*, R162*, R169*, R172*: device TR808clone:R-EU_0207/5V -> TR808clone:R-EU_0207/7
- R59*1: device TR808clone:R-EU_0207/2V -> TR808clone:R-EU_0207/5V
Connections:
- removed net +5V: U$1.+5V, U$2.+5V
Changed lines of the file:
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@@
 <parts>
 <part name="R7*" library="TR808clone" deviceset="R-EU_" device="0207/5V" value="10K"/>
-<part name="R11*" library="TR808clone" deviceset="R-EU_" device="0207/5V" value="22K"/>
+<part name="R11*" library="TR808clone" deviceset="R-EU_" device="0207/7" value="22K"/>
 <part name="R16*" library="TR808clone" deviceset="R-EU_" device="0207/5V" value="4K7"/>
 <part name="R2*" library="TR808clone" deviceset="R-EU_" device="0207/5V" value="22K"/>
@@
 <part name="V359" library="supply1" deviceset="GND" device=""/>
 <part name="R8*" library="TR808clone" deviceset="R-EU_" device="0207/5V" value="10K"/>
-<part name="R12*" library="TR808clone" deviceset="R-EU_" device="0207/5V" value="22K"/>
+<part name="R12*" library="TR808clone" deviceset="R-EU_" device="0207/7" value="22K"/>
 <part name="R17*" library="TR808clone" deviceset="R-EU_" device="0207/5V" value="4K7"/>
-<part name="R1*" library="TR808clone" deviceset="R-EU_" device="0207/5V" value="22K"/>
+<part name="R1*" library="TR808clone" deviceset="R-EU_" device="0207/2V" value="22K"/>
 <part name="R131*" library="TR808clone" deviceset="R-EU_" device="0207/5V" value="22K"/>
 <part name="V362" library="supply1" deviceset="GND" device=""/>
@@
 <part name="C60*" library="TR808clone" deviceset="CPOL-EU" device="E2.5-5" value="10/16"/>
 <part name="V365" library="supply1" deviceset="GND" device=""/>
-<part name="R133*" library="TR808clone" deviceset="R-EU_" device="0207/5V" value="10K"/>
-<part name="R134*" library="TR808clone" deviceset="R-EU_" device="0207/5V" value="100K"/>
+<part name="R133*" library="TR808clone" deviceset="R-EU_" device="0207/7" value="10K"/>
+<part name="R134*" library="TR808clone" deviceset="R-EU_" device="0207/7" value="100K"/>
 <part name="R135*" library="TR808clone" deviceset="R-EU_" device="0207/5V" value="10K"/>
 <part name="R137*" library="TR808clone" deviceset="R-EU_" device="0207/5V" value="470R"/>
@@
 <part name="C63*" library="TR808clone" deviceset="CPOL-EU" device="E2.5-5" value=".47/50"/>
 <part name="V374" library="supply1" deviceset="GND" device=""/>
-<part name="C67*" library="TR808clone" deviceset="C-EU" device="4MM_PITCH" value="22n"/>
+<part name="C67*" library="TR808clone" deviceset="C-EU" device="050-024X044" value="22n"/>
 <part name="V375" library="supply1" deviceset="GND" device=""/>
 <part name="V376" library="supply1" deviceset="GND" device=""/>
-<part name="R145*" library="TR808clone" deviceset="R-EU_" device="0207/5V" value="100R"/>
+<part name="R145*" library="TR808clone" deviceset="R-EU_" device="0207/7" value="100R"/>
 <part name="R152*" library="TR808clone" deviceset="R-EU_" device="0207/5V" value="100R"/>
 <part name="R150*" library="TR808clone" deviceset="R-EU_" device="0207/5V" value="2M"/>
-<part name="D13*" library="TR808clone" deviceset="1N4148" device="DO35-7"/>
-<part name="D14*" library="TR808clone" deviceset="1N4148" device="DO35-7"/>
+<part name="D13*" library="TR808clone" deviceset="1N4148" device="DO35-10" value="1N4148DO35-10"/>
+<part name="D14*" library="TR808clone" deviceset="1N4148" device="DO35-10" value="1N4148DO35-10"/>
 <part name="C65*" library="TR808clone" deviceset="C-EU" device="3.5MM_PITCH" value="1.5n"/>
 <part name="C70*" library="TR808clone" deviceset="C-EU" device="3.5MM_PITCH" value="1.5n"/>
@@
 <part name="C66*" library="TR808clone" deviceset="C-EU" device="3.5MM_PITCH" value="1.5n"/>
 <part name="C72*" library="TR808clone" deviceset="C-EU" device="3.5MM_PITCH" value="1n"/>
-<part name="C68*" library="TR808clone" deviceset="C-EU" device="3.5MM_PITCH" value="1.5n"/>
+<part name="C68*" library="TR808clone" deviceset="C-EU" device="050-024X044" value="1.5n"/>
 <part name="C73*" library="TR808clone" deviceset="C-EU" device="3.5MM_PITCH" value="1n"/>
 <part name="R147*" library="TR808clone" deviceset="R-EU_" device="0207/7" value="2K7"/>
 <part name="R153*" library="rcl" deviceset="R-US_" device="0207/5V" value="2K7"/>
-<part name="R146*" library="TR808clone" deviceset="R-EU_" device="0207/5V" value="68K"/>
+<part name="R146*" library="TR808clone" deviceset="R-EU_" device="0207/7" value="68K"/>
 <part name="R155*" library="TR808clone" deviceset="R-EU_" device="0207/5V" value="68K"/>
 <part name="V383" library="supply1" deviceset="GND" device=""/>
 <part name="V384" library="supply1" deviceset="GND" device=""/>
 <part name="C80*" library="TR808clone" deviceset="C-EU" device="3.5MM_PITCH" value="470p"/>
-<part name="C74*" library="TR808clone" deviceset="C-EU" device="3.5MM_PITCH" value="470p"/>
+<part name="C74*" library="TR808clone" deviceset="C-EU" device="050-025X075" value="470p"/>
 <part name="R160*" library="TR808clone" deviceset="R-EU_" device="0207/5V" value="39K"/>
-<part name="R162*" library="TR808clone" deviceset="R-EU_" device="0207/5V" value="33K"/>
+<part name="R162*" library="TR808clone" deviceset="R-EU_" device="0207/7" value="33K"/>
 <part name="R158*" library="TR808clone" deviceset="R-EU_" device="0207/5V" value="47K"/>
 <part name="R157*" library="TR808clone" deviceset="R-EU_" device="0207/5V" value="47K"/>
 <part name="V389" library="supply1" deviceset="GND" device=""/>
 <part name="V390" library="supply1" deviceset="GND" device=""/>
-<part name="R159*" library="TR808clone" deviceset="R-EU_" device="0207/5V" value="470K"/>
+<part name="R159*" library="TR808clone" deviceset="R-EU_" device="0207/2V" value="470K"/>
 <part name="C81*" library="TR808clone" deviceset="CPOL-EU" device="E2-5" value="33/6.3"/>
 <part name="C79*" library="TR808clone" deviceset="C-EU" device="025-025X050" value="220p"/>
-<part name="R169*" library="TR808clone" deviceset="R-EU_" device="0207/5V" value="1K"/>
+<part name="R169*" library="TR808clone" deviceset="R-EU_" device="0207/7" value="1K"/>
 <part name="R161*" library="TR808clone" deviceset="R-EU_" device="0207/2V" value="470K"/>
 <part name="C83*" library="TR808clone" deviceset="CPOL-EU" device="E2-5" value="33/6.3"/>
 <part name="C82*" library="TR808clone" deviceset="C-EU" device="025-025X050" value="220p"/>
-<part name="R172*" library="TR808clone" deviceset="R-EU_" device="0207/5V" value="1K"/>
+<part name="R172*" library="TR808clone" deviceset="R-EU_" device="0207/7" value="1K"/>
 <part name="R132*" library="TR808clone" deviceset="R-EU_" device="0207/5V" value="100K"/>
 <part name="R140*" library="TR808clone" deviceset="R-EU_" device="0207/5V" value="33K"/>
-<part name="R156*" library="TR808clone" deviceset="R-EU_" device="0207/5V" value="22K"/>
+<part name="R156*" library="TR808clone" deviceset="R-EU_" device="0207/7" value="22K"/>
 <part name="R154*" library="TR808clone" deviceset="R-EU_" device="0207/5V" value="22K"/>
 <part name="R144*" library="TR808clone" deviceset="R-EU_" device="0207/5V" value="33K"/>
@@
 <part name="OH_LEVEL" library="pot" deviceset="3RP/1610N" device="" value="100KA"/>
 <part name="DECAY" library="pot" deviceset="3RP/1610N" device="" value="2MB"/>
-<part name="R142*" library="TR808clone" deviceset="R-EU_" device="0207/5V" value="33K"/>
+<part name="R142*" library="TR808clone" deviceset="R-EU_" device="0207/7" value="33K"/>
 <part name="V44" library="supply1" deviceset="GND" device=""/>
 <part name="V45" library="supply1" deviceset="GND" device=""/>
@@
 <part name="R55*1" library="TR808clone" deviceset="R-EU_" device="0207/5V" value="22K"/>
 <part name="V2" library="supply1" deviceset="GND" device=""/>
-<part name="C15*1" library="TR808clone" deviceset="C-EU" device="3.5MM_PITCH" value="3.3n"/>
+<part name="C15*1" library="TR808clone" deviceset="C-EU" device="050-024X044" value="3.3n"/>
 <part name="C16*1" library="TR808clone" deviceset="C-EU" device="3.5MM_PITCH" value="3.3n"/>
 <part name="V3" library="supply1" deviceset="GND" device=""/>
-<part name="R59*1" library="TR808clone" deviceset="R-EU_" device="0207/2V" value="82K"/>
+<part name="R59*1" library="TR808clone" deviceset="R-EU_" device="0207/5V" value="82K"/>
 <part name="R58*1" library="TR808clone" deviceset="R-EU_" device="0207/2V" value="560R"/>
 <part name="IC1" library="linear" deviceset="TL072" device="P"/>
@@
 <part name="P-1" library="supply1" deviceset="-12V" device=""/>
 <part name="V14" library="supply1" deviceset="GND" device=""/>
-<part name="P+2" library="supply1" deviceset="+5V" device=""/>
 <part name="CH_ACCENT" library="solpad" deviceset="LSP11" device=""/>
 <part name="CH_TRIG" library="solpad" deviceset="LSP11" device=""/>
@@
 <part name="P-4" library="supply1" deviceset="-12V" device=""/>
 <part name="V4" library="supply1" deviceset="GND" device=""/>
-<part name="P+4" library="supply1" deviceset="+5V" device=""/>
 <part name="Q1" library="808_lt" deviceset="2N3904" device=""/>
 <part name="Q2" library="808_lt" deviceset="2N3904" device=""/>
@@
 <instance part="P-1" gate="1" x="-81.28" y="81.28"/>
 <instance part="V14" gate="1" x="-68.58" y="96.52"/>
-<instance part="P+2" gate="1" x="-76.2" y="111.76"/>
 <instance part="IC1" gate="A" x="147.32" y="48.26" rot="MR180"/>
 <instance part="IC1" gate="B" x="147.32" y="7.62" rot="MR180"/>
@@
 <instance part="P-4" gate="1" x="-81.28" y="7.62"/>
 <instance part="V4" gate="1" x="-68.58" y="22.86"/>
-<instance part="P+4" gate="1" x="-76.2" y="38.1"/>
 <instance part="Q1" gate="G1" x="104.14" y="55.88"/>
 <instance part="Q2" gate="G1" x="104.14" y="15.24"/>
@@
 </segment>
 </net>
-<net name="+5V" class="0">
-<segment>
-<pinref part="U$1" gate="G$1" pin="+5V"/>
-<pinref part="P+2" gate="1" pin="+5V"/>
-<wire x1="-86.36" y1="96.52" x2="-76.2" y2="96.52" width="0.1524" layer="91"/>
-<wire x1="-76.2" y1="96.52" x2="-76.2" y2="109.22" width="0.1524" layer="91"/>
-</segment>
-<segment>
-<pinref part="U$2" gate="G$1" pin="+5V"/>
-<pinref part="P+4" gate="1" pin="+5V"/>
-<wire x1="-86.36" y1="22.86" x2="-76.2" y2="22.86" width="0.1524" layer="91"/>
-<wire x1="-76.2" y1="22.86" x2="-76.2" y2="35.56" width="0.1524" layer="91"/>
-</segment>
-</net>

Commit message: 94pct ar
Parts:
- R130*, R140*, R173*: device TR808clone:R-EU_0207/5V -> TR808clone:R-EU_0207/7
- R145*, R162*: device TR808clone:R-EU_0207/7 -> TR808clone:R-EU_0207/5V
Changed lines of the file:
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@@
 <part name="V362" library="supply1" deviceset="GND" device=""/>
 <part name="V363" library="supply1" deviceset="GND" device=""/>
-<part name="R130*" library="TR808clone" deviceset="R-EU_" device="0207/5V" value="10K"/>
+<part name="R130*" library="TR808clone" deviceset="R-EU_" device="0207/7" value="10K"/>
 <part name="V364" library="supply1" deviceset="GND" device=""/>
 <part name="C60*" library="TR808clone" deviceset="CPOL-EU" device="E2.5-5" value="10/16"/>
@@
 <part name="R136*" library="TR808clone" deviceset="R-EU_" device="0207/5V" value="100R"/>
 <part name="R141*" library="TR808clone" deviceset="R-EU_" device="0207/5V" value="33K"/>
-<part name="R173*" library="TR808clone" deviceset="R-EU_" device="0207/5V" value="330K"/>
+<part name="R173*" library="TR808clone" deviceset="R-EU_" device="0207/7" value="330K"/>
 <part name="C63*" library="TR808clone" deviceset="CPOL-EU" device="E2.5-5" value=".47/50"/>
 <part name="V374" library="supply1" deviceset="GND" device=""/>
@@
 <part name="V375" library="supply1" deviceset="GND" device=""/>
 <part name="V376" library="supply1" deviceset="GND" device=""/>
-<part name="R145*" library="TR808clone" deviceset="R-EU_" device="0207/7" value="100R"/>
+<part name="R145*" library="TR808clone" deviceset="R-EU_" device="0207/5V" value="100R"/>
 <part name="R152*" library="TR808clone" deviceset="R-EU_" device="0207/5V" value="100R"/>
 <part name="R150*" library="TR808clone" deviceset="R-EU_" device="0207/5V" value="2M"/>
@@
 <part name="C74*" library="TR808clone" deviceset="C-EU" device="050-025X075" value="470p"/>
 <part name="R160*" library="TR808clone" deviceset="R-EU_" device="0207/5V" value="39K"/>
-<part name="R162*" library="TR808clone" deviceset="R-EU_" device="0207/7" value="33K"/>
+<part name="R162*" library="TR808clone" deviceset="R-EU_" device="0207/5V" value="33K"/>
 <part name="R158*" library="TR808clone" deviceset="R-EU_" device="0207/5V" value="47K"/>
 <part name="R157*" library="TR808clone" deviceset="R-EU_" device="0207/5V" value="47K"/>
@@
 <part name="R172*" library="TR808clone" deviceset="R-EU_" device="0207/7" value="1K"/>
 <part name="R132*" library="TR808clone" deviceset="R-EU_" device="0207/5V" value="100K"/>
-<part name="R140*" library="TR808clone" deviceset="R-EU_" device="0207/5V" value="33K"/>
+<part name="R140*" library="TR808clone" deviceset="R-EU_" device="0207/7" value="33K"/>
 <part name="R156*" library="TR808clone" deviceset="R-EU_" device="0207/7" value="22K"/>
 <part name="R154*" library="TR808clone" deviceset="R-EU_" device="0207/5V" value="22K"/>
